File: Projeto1/projeto1/projeto1.brd (EAGLE design)
At the start: 122.9 x 59.7 mm, 2 parts

Commit message: Add files via upload
Parts:
- removed U$1: DEVICE1, Cactus_Library:DEVICE_FOOTPRINT
- added U$2: DEVICE1, Cactus_Library:DEVICE_FOOTPRINT
- moved BOARD1 20.4 mm to (55.9, 16.5), turned to 0 degrees
Connections:
- net GND: now also U$2.GND; no longer U$1.GND
- net N$1: now also U$2.SDA; no longer U$1.SDA
- net N$2: now also BOARD1.D5, U$2.CSB; no longer BOARD1.D19, U$1.SDO
- net N$3: now also BOARD1.D19, U$2.SDO; no longer BOARD1.D18, U$1.SCL
- net N$5: now also BOARD1.D18, U$2.SCL; no longer BOARD1.D5, U$1.CSB
- net VCC: now also U$2.VCC; no longer U$1.VCC
Routing:
- net VCC: track 0.00 -> 181.8 mm
- net N$1: track 0.00 -> 85.0 mm
- net N$3: track 0.00 -> 72.1 mm
- net N$5: track 0.00 -> 66.5 mm
- net N$2: track 0.00 -> 62.5 mm
- added copper zone on layer 16, net GND
Changed lines of the file:
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@@
 <layer number="45" name="Holes" color="7" fill="1" visible="yes" active="yes"/>
 <layer number="46" name="Milling" color="3" fill="1" visible="no" active="yes"/>
-<layer number="47" name="Measures" color="7" fill="1" visible="no" active="yes"/>
+<layer number="47" name="Measures" color="7" fill="1" visible="yes" active="yes"/>
 <layer number="48" name="Document" color="7" fill="1" visible="yes" active="yes"/>
 <layer number="49" name="Reference" color="7" fill="1" visible="yes" active="yes"/>
@@
 <wire x1="119.05" y1="49.52" x2="-3.81" y2="49.52" width="0" layer="20"/>
 <wire x1="-3.81" y1="49.52" x2="-3.81" y2="-10.16" width="0" layer="20"/>
+<hole x="-1.27" y="46.99" drill="3"/>
+<hole x="116.84" y="46.99" drill="3"/>
+<hole x="116.84" y="-7.62" drill="3"/>
+<hole x="-1.27" y="-7.62" drill="3"/>
+<dimension x1="-3.81" y1="-12.7" x2="119.38" y2="-12.7" x3="57.785" y3="-15.24" textsize="1.778" layer="47"/>
+<dimension x1="123.19" y1="-10.16" x2="123.19" y2="49.53" x3="125.73" y3="19.685" textsize="1.778" layer="47"/>
 </plain>
 <attributes>
@@
 <param name="mdDrill" value="6mil"/>
 <param name="mdSmdStop" value="0mil"/>
-<param name="msWidth" value="50mil"/>
-<param name="msDrill" value="0.35mm"/>
+<param name="msWidth" value="1.7mm"/>
+<param name="msDrill" value="1mm"/>
 <param name="msMicroVia" value="9.99mm"/>
 <param name="msBlindViaRatio" value="0.5"/>
@@
 <param name="rvMicroViaOuter" value="0.25"/>
 <param name="rvMicroViaInner" value="0.25"/>
-<param name="rlMinPadTop" value="10mil"/>
-<param name="rlMaxPadTop" value="20mil"/>
+<param name="rlMinPadTop" value="22mil"/>
+<param name="rlMaxPadTop" value="30mil"/>
 <param name="rlMinPadInner" value="10mil"/>
 <param name="rlMaxPadInner" value="20mil"/>
-<param name="rlMinPadBottom" value="10mil"/>
-<param name="rlMaxPadBottom" value="20mil"/>
-<param name="rlMinViaOuter" value="8mil"/>
-<param name="rlMaxViaOuter" value="20mil"/>
-<param name="rlMinViaInner" value="8mil"/>
-<param name="rlMaxViaInner" value="20mil"/>
+<param name="rlMinPadBottom" value="22mil"/>
+<param name="rlMaxPadBottom" value="30mil"/>
+<param name="rlMinViaOuter" value="22mil"/>
+<param name="rlMaxViaOuter" value="22mil"/>
+<param name="rlMinViaInner" value="10mil"/>
+<param name="rlMaxViaInner" value="10mil"/>
 <param name="rlMinMicroViaOuter" value="4mil"/>
 <param name="rlMaxMicroViaOuter" value="20mil"/>
@@
 </autorouter>
 <elements>
-<element name="U$1" library="Cactus_Library" package="DEVICE_FOOTPRINT" value="DEVICE1" x="21.59" y="20.32" smashed="yes" rot="R90"/>
-<element name="BOARD1" library="ESP32-DEVKITV1" package="ESP32-DEVKITV1" value="ESP32DEVKITV1" x="54.61" y="36.83" smashed="yes" rot="R270">
-<attribute name="ESP32-DEVKITV1" value="" x="54.61" y="36.83" size="1.778" layer="27" rot="R270" display="off"/>
-<attribute name="NAME" x="82.82" y="44.1" size="1.27" layer="21" rot="R270"/>
+<element name="BOARD1" library="ESP32-DEVKITV1" package="ESP32-DEVKITV1" value="ESP32DEVKITV1" x="55.88" y="16.51" smashed="yes">
+<attribute name="ESP32-DEVKITV1" value="" x="55.88" y="16.51" size="1.778" layer="27" display="off"/>
+<attribute name="NAME" x="48.61" y="44.72" size="1.27" layer="21"/>
 </element>
+<element name="U$2" library="Cactus_Library" package="DEVICE_FOOTPRINT" value="DEVICE1" x="20.32" y="21.59" smashed="yes" rot="R90"/>
 </elements>
 <signals>
 <signal name="GND">
-<contactref element="U$1" pad="GND"/>
 <contactref element="BOARD1" pad="GND"/>
-<wire x1="29.21" y1="29.21" x2="80.01" y2="34.29" width="0" layer="19" extent="1-1"/>
+<contactref element="U$2" pad="GND"/>
+<polygon width="1.7" layer="16">
+<vertex x="-3.81" y="49.53"/>
+<vertex x="118.11" y="49.53"/>
+<vertex x="119.38" y="48.26"/>
+<vertex x="119.38" y="-8.89"/>
+<vertex x="118.11" y="-10.16"/>
+<vertex x="-3.81" y="-10.16"/>
+</polygon>
+<wire x1="27.94" y1="30.48" x2="58.42" y2="41.91" width="0" layer="19" extent="1-1"/>
 </signal>
 <signal name="N$1">
-<contactref element="U$1" pad="SDA"/>
 <contactref element="BOARD1" pad="D23"/>
-<wire x1="29.21" y1="13.97" x2="54.61" y2="1.27" width="0" layer="19" extent="1-1"/>
+<contactref element="U$2" pad="SDA"/>
+<wire x1="27.94" y1="15.24" x2="28.8412" y2="14.3388" width="1.7" layer="16"/>
+<wire x1="28.8412" y1="14.3388" x2="29.14486875" y2="14.3388" width="1.7" layer="16"/>
+<wire x1="29.14486875" y1="14.3388" x2="30.8488" y2="12.63486875" width="1.7" layer="16"/>
+<wire x1="30.8488" y1="12.63486875" x2="30.8488" y2="12.3312" width="1.7" layer="16"/>
+<wire x1="30.8488" y1="12.3312" x2="45.72" y2="-2.54" width="1.7" layer="16"/>
+<wire x1="45.72" y1="-2.54" x2="82.55" y2="-2.54" width="1.7" layer="16"/>
+<wire x1="82.55" y1="-2.54" x2="91.8088" y2="6.7188" width="1.7" layer="16"/>
+<wire x1="91.8088" y1="6.7188" x2="91.8088" y2="16.51" width="1.7" layer="16"/>
+<wire x1="91.8088" y1="16.51" x2="91.44" y2="16.51" width="0" layer="19" extent="16-16"/>
 </signal>
 <signal name="N$5">
-<contactref element="U$1" pad="CSB"/>
+<contactref element="U$2" pad="SCL"/>
+<contactref element="BOARD1" pad="D18"/>
+<wire x1="76.2" y1="16.51" x2="76.2" y2="6.35" width="1.7" layer="16"/>
+<wire x1="76.2" y1="6.35" x2="74.93" y2="5.08" width="1.7" layer="16"/>
+<wire x1="74.93" y1="5.08" x2="45.7367625" y2="5.08" width="1.7" layer="16"/>
+<wire x1="36.2488" y1="14.5679625" x2="36.2488" y2="14.87163125" width="1.7" layer="16"/>
+<wire x1="36.2488" y1="14.87163125" x2="28.26043125" y2="22.86" width="1.7" layer="16"/>
+<wire x1="28.26043125" y1="22.86" x2="27.94" y2="22.86" width="1.7" layer="16"/>
+<wire x1="45.7367625" y1="5.08" x2="36.2488" y2="14.5679625" width="1.7" layer="16"/>
+</signal>
+<signal name="N$2">
+<contactref element="U$2" pad="CSB"/>
 <contactref element="BOARD1" pad="D5"/>
-<wire x1="29.21" y1="21.59" x2="54.61" y2="19.05" width="0" layer="19" extent="1-1"/>
-</signal>
-<signal name="N$2">
-<contactref element="U$1" pad="SDO"/>
+<wire x1="73.66" y1="16.51" x2="73.66" y2="7.62" width="1.7" layer="16"/>
+<wire x1="46.99" y1="7.62" x2="27.94" y2="26.67" width="1.7" layer="16"/>
+<wire x1="73.66" y1="7.62" x2="46.99" y2="7.62" width="1.7" layer="16"/>
+</signal>
+<signal name="N$3">
+<contactref element="U$2" pad="SDO"/>
 <contactref element="BOARD1" pad="D19"/>
-<wire x1="29.21" y1="25.4" x2="54.61" y2="13.97" width="0" layer="19" extent="1-1"/>
-</signal>
-<signal name="N$3">
-<contactref element="U$1" pad="SCL"/>
-<contactref element="BOARD1" pad="D18"/>
-<wire x1="29.21" y1="17.78" x2="54.61" y2="16.51" width="0" layer="19" extent="1-1"/>
+<wire x1="27.94" y1="19.05" x2="28.8412" y2="18.1488" width="1.7" layer="16"/>
+<wire x1="33.5488" y1="13.75325" x2="33.5488" y2="13.44958125" width="1.7" layer="16"/>
+<wire x1="28.8412" y1="18.1488" x2="29.15325" y2="18.1488" width="1.7" layer="16"/>
+<wire x1="29.15325" y1="18.1488" x2="33.5488" y2="13.75325" width="1.7" layer="16"/>
+<wire x1="45.72838125" y1="1.27" x2="76.2" y2="1.27" width="1.7" layer="16"/>
+<wire x1="76.2" y1="1.27" x2="78.74" y2="3.81" width="1.7" layer="16"/>
+<wire x1="78.74" y1="3.81" x2="78.74" y2="12.7" width="1.7" layer="16"/>
+<wire x1="78.74" y1="12.7" x2="78.74" y2="14.93633125" width="1.7" layer="16"/>
+<wire x1="33.5488" y1="13.44958125" x2="45.72838125" y2="1.27" width="1.7" layer="16"/>
+<wire x1="78.74" y1="16.51" x2="78.74" y2="14.93633125" width="1.7" layer="16"/>
 </signal>
 <signal name="VCC">
-<contactref element="U$1" pad="VCC"/>
 <contactref element="BOARD1" pad="VIN"/>
-<wire x1="80.01" y1="36.83" x2="29.21" y2="10.16" width="0" layer="19" extent="1-1"/>
+<contactref element="U$2" pad="VCC"/>
+<wire x1="27.94" y1="11.43" x2="28.1488" y2="11.2212" width="1.7" layer="16"/>
+<wire x1="28.1488" y1="11.2212" x2="28.1488" y2="11.21281875" width="1.7" layer="16"/>
+<wire x1="44.60161875" y1="-5.24" x2="44.61" y2="-5.24" width="1.7" layer="16"/>
+<wire x1="44.61" y1="-5.24" x2="45.72" y2="-6.35" width="1.7" layer="16"/>
+<wire x1="28.1488" y1="11.21281875" x2="44.60161875" y2="-5.24" width="1.7" layer="16"/>
+<wire x1="45.72" y1="-6.35" x2="100.33" y2="-6.35" width="1.7" layer="16"/>
+<wire x1="100.33" y1="-6.35" x2="102.87" y2="-3.81" width="1.7" layer="16"/>
+<wire x1="102.87" y1="-3.81" x2="102.87" y2="44.45" width="1.7" layer="16"/>
+<wire x1="102.87" y1="44.45" x2="101.6" y2="45.72" width="1.7" layer="16"/>
+<wire x1="55.5112" y1="43.11486875" x2="55.5112" y2="41.91" width="1.7" layer="16"/>
+<wire x1="101.6" y1="45.72" x2="58.11633125" y2="45.72" width="1.7" layer="16"/>
+<wire x1="58.11633125" y1="45.72" x2="55.5112" y2="43.11486875" width="1.7" layer="16"/>
+<wire x1="55.5112" y1="41.91" x2="55.88" y2="41.91" width="0" layer="19" extent="16-16"/>
 </signal>
 </signals>
